Commit message: modified dimensions due to CAD model

File: robot_models/fugu-c.urdf (robot description, URDF)
Before this commit: robot fugu-c, 5 links, 4 joints
Links:
- link base_link: geometry visual cylinder length=0.208 radius=0.106
Joints:
- joint base_link_to_stereo_down: origin xyz=0 0 0.1 rpy=0 -1.5708 0 -> xyz=0 0 0.095 rpy=0 -1.5708 0
- joint base_link_to_stereo_forward: origin xyz=0.1 0 0 rpy=3.1416 0 0 -> xyz=0.094 0 0 rpy=3.1416 0 0
